File: tp4potencia.kicad_sch (KiCad schematic)
At the start: 36 parts, among them J1 Screw_Terminal_01x02, J2 Screw_Terminal_01x03, J3 Screw_Terminal_01x02, Q1 IRF840, Q2 IRF840, SW1 SW_SPST_Lamp, SW2 SW_SPDT, SW4 SW_SPDT, T1 Trafo1, U1 LTV-817, U4 LM339

Commit message: Ver 1.0
Parts:
- R2: value 10K -> 150; Power 1/4W -> 2W
